Commit message: tested for params

File: usv_sim/xacro/diffboat.xacro (robot description, xacro)
@@ -30,5 +30,5 @@
             <switchService>switch</switchService>
             <updateRate>100</updateRate>
-            <link>fwd_left</link>
+            <link>${robotName}/fwd_left</link>
             <thruster>
 				<effortUnderWater>11.5</effortUnderWater>
