Commit message: motion vertical and external force with D control

File: usv_sim/xacro/boat_subdivided_validated.xacro (robot description, xacro)
@@ -396,5 +396,9 @@
         </inertial>
     </link>
-    <gazebo reference="hokuyo_link">
+        <!-- Noise parameters based on published spec for Hokuyo laser
+        achieving "+-30mm" accuracy at range < 10m.  A mean of 0.0m and
+        stddev of 0.01m will put 99.7% of samples within 0.03m of the true
+        reading. -->
+  <!-- <gazebo reference="hokuyo_link">
         <sensor type="gpu_ray" name="head_hokuyo_sensor">
         <pose>0 0 0 0 0 0</pose>
@@ -417,8 +421,4 @@
         <noise>
         <type>gaussian</type>
-        <!-- Noise parameters based on published spec for Hokuyo laser
-        achieving "+-30mm" accuracy at range < 10m.  A mean of 0.0m and
-        stddev of 0.01m will put 99.7% of samples within 0.03m of the true
-        reading. -->
         <mean>0.0</mean>
         <stddev>0.01</stddev>
@@ -430,4 +430,4 @@
         </plugin>
         </sensor>
-    </gazebo>
+    </gazebo> -->
 </xacro>

File: usv_sim/xacro/diffboat.xacro (robot description, xacro)
@@ -1,4 +1,6 @@
 <?xml version="1.0"?>
 <robot name="diffboat" xmlns:xacro="http://www.ros.org/wiki/xacro">
+    <xacro:arg name="robotName" default="diffboat" />
+    <xacro:property name="robotName" value="$(arg robotName)" />
     <xacro:arg name="windType" default="global" />
     <xacro:arg name="waterType" default="global" />
@@ -9,4 +11,18 @@
     <xacro:property name="extraPayload" value="3" />
     <xacro:include filename="$(find usv_sim)/xacro/boat_subdivided_validated.xacro" />
+    <!-- todo
+    1. change name
+    2. inside robot namespace -->
+    <!-- planar move plugin for cmd_vel control -->
+    <!-- <gazebo>
+        <plugin name="object_controller" filename="libgazebo_ros_planar_move.so">
+        <commandTopic>cmd_vel</commandTopic>
+        <odometryTopic>odom</odometryTopic>
+        <odometryFrame>${robotName}/odometry</odometryFrame>
+        <odometryRate>20.0</odometryRate>
+        <robotBaseFrame>${robotName}/test</robotBaseFrame>
+        <robotNamespace>${robotName}</robotNamespace>
+        </plugin>
+    </gazebo> -->
     <!-- Plugin list -->
     <gazebo>
@@ -27,14 +43,4 @@
         </plugin>
     </gazebo>
-    <gazebo>
-        <plugin name="object_controller" filename="libgazebo_ros_planar_move.so">
-        <commandTopic>cmd_vel</commandTopic>
-        <odometryTopic>odom</odometryTopic>
-        <odometryFrame>odom</odometryFrame>
-        <odometryRate>20.0</odometryRate>
-        <robotBaseFrame>base_link</robotBaseFrame>
-        <robotNamespace>diffboat</robotNamespace>
-        </plugin>
-    </gazebo>
     <!-- Define two steering thrusters, with assumed force control in Z-direction -->
     <xacro:thruster_link name="fwd_left"  xyz="-0.3 0 -0.1" rpy="0 ${-PI/2-0.26} 0" rotationAxis="1 0 0" lowerLimit="0" upperLimit="0" parentLink="back_l_link"/>

Commit message: save for testing

File: usv_sim/xacro/boat_subdivided_validated.xacro (robot description, xacro)
@@ -9,5 +9,7 @@
     <xacro:property name="middle_water_displaced_mass" value="10"/>
     <xacro:property name="front_water_displaced_mass" value="5"/>
-    <xacro:property name="scale" value="0.21"/>
+    <!-- <xacro:property name="scale" value="0.21"/> -->
+    <xacro:arg name="scale" default="0.21" />
+    <xacro:property name="scale" value="$(arg scale)" />
     <xacro:property name="bl1" value=".1" />
     <xacro:property name="bl2" value=".1" />

File: usv_sim/xacro/diffboat.xacro (robot description, xacro)
@@ -3,4 +3,6 @@
     <xacro:arg name="robotName" default="diffboat" />
     <xacro:property name="robotName" value="$(arg robotName)" />
+    <xacro:arg name="scale" default="0.21" />
+    <xacro:property name="scale" value="$(arg scale)" />
     <xacro:arg name="windType" default="global" />
     <xacro:arg name="waterType" default="global" />

Commit message: test setup save for IROS

File: usv_sim/xacro/boat_subdivided_validated.xacro (robot description, xacro)
@@ -372,5 +372,5 @@
     <!-- Sensors -->
     <!-- Hokuyo Laser -->
-    <joint name="hokuyo_joint" type="revolute">
+    <!-- <joint name="hokuyo_joint" type="revolute">
         <axis xyz="0 1 0" />
         <origin xyz="0.50 0 0.15" rpy="0 0 0"/>
@@ -397,5 +397,5 @@
         <inertia ixx="1e-6" ixy="0" ixz="0" iyy="1e-6" iyz="0" izz="1e-6" />
         </inertial>
-    </link>
+    </link> -->
         <!-- Noise parameters based on published spec for Hokuyo laser
         achieving "+-30mm" accuracy at range < 10m.  A mean of 0.0m and
